File: demo32.sch (KiCad schematic (older format))
At the start: 198 parts, among them J10 LIPO_1x2, J101 ANALOG_IN1, J102 ANALOG_IN2, J103 ANALOG_OUT1, J104 ANALOG_OUT2, J105 SERIAL_IO_1x4, J106 EXPANSION_IO_1x9, J107 RELAY_CONTACTS_1x9, J108 EX_PWR_IN_1x4, J109 SPI_PORT_1x6, J8 Micro_SD_Card_Det, J9 USB_MICRO_AB, K101 G6K-2, Q1 DMP2160UW, SW1 RESET, SW102 USER, SW103 BOOT, SW110 RED, SW111 GREEN, SW112 YELLOW, SW113 BLUE, SW3 BLACK, SW4 BLACK, U1 STM32F405RGTx, U101 MR25H10, U102 ULN2003A, U2 MCP1703, U3 MMA7660, U4 MIC2005A-1YM5, Y1 12MHz, Y2 32.768kHz

Commit message: documentation cleanup, one local project library
Parts:
- A101: footprint .novac:MODULE_OLED_910 -> .demo32:MODULE_OLED_910; symbol .novac:ASSY_OLED_910MILS_128x32_I2C -> .demo32:ASSY_OLED_910MILS_128x32_I2C
- BT101: footprint .novac:BatteryHolder_Keystone_1059_1x2032 -> .demo32:BatteryHolder_Keystone_1059_1x2032; symbol .novac:Battery_Cell -> .demo32:Battery_Cell
- C1, C104, C106, C11, C12, C13, C2, C3, C4, C5, C6, C8, C9: footprint .novac:C_0805_2012Metric -> .demo32:C_0805_2012Metric; symbol .novac:C_SMALL -> .demo32:C_SMALL
- C10, C16, C17, C18, C19, C20, C7: footprint .novac:C_0805_2012Metric -> .demo32:C_0805_2012Metric; symbol .novac:C2_SMALL -> .demo32:C2_SMALL
- D1: footprint .novac:LED_0805_2012Metric_LiteOn_C171 -> .demo32:LED_0805_2012Metric_LiteOn_C171; symbol .novac:DIODE -> .demo32:DIODE
- D2, D3, D4, D5: footprint .novac:LED_0805_2012Metric_LiteOn_C171 -> .demo32:LED_0805_2012Metric_LiteOn_C171; symbol .novac:LED -> .demo32:LED
- H1, H2, H3, H4: footprint .novac:MountingHole_3.2mm_M3_ISO7380_Pad -> .demo32:MountingHole_3.2mm_M3_ISO7380_Pad; symbol .novac:MountingHole_Pad -> .demo32:MountingHole_Pad
- J10: footprint .novac:TE_640454-2-FLIP -> .demo32:TE_640454-2-FLIP; symbol .novac:IO_JACK_M02 -> .demo32:IO_JACK_M02
- J101, J102, J103, J104: footprint .novac:BNC_TEConnectivity_1634503_Vertical -> .demo32:BNC_TEConnectivity_1634503_Vertical
- J105: footprint .novac:TE_640454-4 -> .demo32:TE_640454-4; symbol .novac:IO_JACK_M04 -> .demo32:IO_JACK_M04
- J106, J107: footprint .novac:TE_640454-9 -> .demo32:TE_640454-9; symbol .novac:IO_JACK_M09 -> .demo32:IO_JACK_M09
- J108: footprint .novac:TE_640454-4_FLIP -> .demo32:TE_640454-4_FLIP; symbol .novac:IO_JACK_M04 -> .demo32:IO_JACK_M04
- J109: footprint .novac:TE_640454-6 -> .demo32:TE_640454-6; symbol .novac:IO_JACK_M06 -> .demo32:IO_JACK_M06
- J8: footprint .novac:microSD_HC_Hirose_DM3BT-DSF-PEJS -> .demo32:microSD_HC_Hirose_DM3BT-DSF-PEJS; symbol .novac:Micro_SD_Card_Det -> .demo32:Micro_SD_Card_Det
- J9: footprint .novac:USB_Micro-AB_Molex_47590-0001 -> .demo32:USB_Micro-AB_Molex_47590-0001; symbol .novac:USB_B_Micro -> .demo32:USB_B_Micro
- K101: footprint .novac:Relay_DPDT_Omron_G6K-2F -> .demo32:Relay_DPDT_Omron_G6K-2F; symbol .novac:G6K-2 -> .demo32:G6K-2
- L1: footprint .novac:L_0805_2012Metric -> .demo32:L_0805_2012Metric
- LOGO1: footprint .novac:OSHW-Logo2_7.3x6mm_SilkScreen -> .demo32:OSHW-Logo2_7.3x6mm_SilkScreen; symbol .novac:Logo_Open_Hardware_Large -> .demo32:Logo_Open_Hardware_Large
- Q1: footprint .novac:SOT-23 -> .demo32:SOT-23
- R1, R10, R101, R102, R103, R104, R105, R106, R107, R108, R109, R11, R110, R111, R112, R113, R114, R115, R116, R117, R12, R120, R121, R123, R124, R125, R126, R128, R137, R14, R15, R16, R17, R19, R2, R20, R22, R3, R4, R5, R6, R7, R8, R9: footprint .novac:R_0805_2012Metric -> .demo32:R_0805_2012Metric; symbol .novac:R_US -> .demo32:R_US
- SW1, SW103, SW110, SW111, SW112, SW113, SW3, SW4: footprint .novac:SW_PUSH_6mm -> .demo32:SW_PUSH_6mm
- SW102: footprint .novac:RotaryEncoder_CTS_11CE -> .demo32:RotaryEncoder_CTS_11CE; symbol .novac:RotaryEncoder_Switch -> .demo32:RotaryEncoder_Switch
- TP10, TP11, TP14, TP15, TP16, TP17, TP2, TP20, TP21, TP22, TP23, TP24, TP25, TP26, TP27, TP28, TP29, TP2A1, TP30, TP33, TP34, TP35, TP36, TP37, TP38, TP39, TP3V3, TP40, TP41, TP46, TP49, TP50, TP51, TP52, TP53, TP54, TP56, TP57, TP58, TP59, TP61, TP62, TP8, TP9, TPGEXT1, TPGLIPO1, TPGND1, TPGND2, TPGND3, TPGND4, TPGND5, TPGND6, TPGND7, TPGND8, TPMV0, TPMV3, TPVBUS5, TPVEXT1, TPVIN5, TPVLIPO1: footprint .novac:TestPoint_Keystone_5000-5004_Miniature -> .demo32:TestPoint_Keystone_5000-5004_Miniature; symbol .novac:TestPoint -> .demo32:TestPoint
- U1: footprint .novac:LQFP-64_10x10mm_P0.5mm -> .demo32:LQFP-64_10x10mm_P0.5mm; symbol .novac:STM32F405RGTx -> .demo32:STM32F405RGTx
- U101: footprint .novac:DFN-8-1EP_6x5mm_P1.27mm_EP2x2mm -> .demo32:DFN-8-1EP_6x5mm_P1.27mm_EP2x2mm; symbol .novac:MR25H10 -> .demo32:MR25H10
- U102: footprint .novac:SOIC-16_3.9x9.9mm_P1.27mm -> .demo32:SOIC-16_3.9x9.9mm_P1.27mm; symbol .novac:ULN2003 -> .demo32:ULN2003
- U2: footprint .novac:SOT-223-3_TabPin2 -> .demo32:SOT-223-3_TabPin2; symbol .novac:MCP1703 -> .demo32:MCP1703
- U3: footprint .novac:DFN-10_3x3mm_P0.5mm -> .demo32:DFN-10_3x3mm_P0.5mm; symbol .novac:MMA7660 -> .demo32:MMA7660
- U4: footprint .novac:SOT-23-5 -> .demo32:SOT-23-5; symbol .novac:MIC2005A-1YM5 -> .demo32:MIC2005A-1YM5
- XR1, XR10, XR11, XR12, XR13, XR14, XR15, XR16, XR17, XR18, XR19, XR2, XR20, XR21, XR22, XR25, XR26, XR3, XR4, XR5, XR6, XR7, XR8, XR9: footprint .novac:MODULE_TRACER -> .demo32:MODULE_TRACER; symbol .novac:TRACER1 -> .demo32:TRACER1
- XR27, XR28, XR29, XR30, XR31, XR32: footprint .novac:MODULE_TRACER -> .demo32:MODULE_TRACER; symbol .novac:TRACER2 -> .demo32:TRACER2
- Y1: footprint .novac:Crystal_SMD_Abracon_ABM7-2Pin_6.0x3.5mm -> .demo32:Crystal_SMD_Abracon_ABM7-2Pin_6.0x3.5mm
- Y2: footprint .novac:Crystal_C26-LF_D2.1mm_L6.5mm_Horizontal_1EP_style1 -> .demo32:Crystal_C26-LF_D2.1mm_L6.5mm_Horizontal_1EP_style1

Commit message: Making BOM
Parts:
- TP10, TP11, TP14, TP15, TP16, TP17, TP2, TP20, TP21, TP22, TP23, TP24, TP25, TP26, TP27, TP28, TP29, TP2A1, TP30, TP33, TP34, TP35, TP36, TP37, TP38, TP39, TP40, TP41, TP46, TP49, TP50, TP51, TP52, TP53, TP54, TP56, TP57, TP58, TP59, TP61, TP62, TP8, TP9: value TestPoint -> TestPointWhite
- TP3V3, TPMV3: value TestPoint -> TestPointRed
- TPGEXT1, TPGLIPO1, TPGND1, TPGND2, TPGND3, TPGND4, TPGND5, TPGND6, TPGND7, TPGND8, TPMV0: value TestPoint -> TestPointBlack
- TPVBUS5, TPVEXT1, TPVIN5, TPVLIPO1: value TestPoint -> TestPointOrange
Other:
- note added: "BK"
- note added: "BLACK"
- note added: "OG"
- note added: "ORANGE"
- note added: "RD"
- note added: "RED"
- note added: "TEST POINT COLOR CODE"
- note added: "WH"
- note added: "WHITE"
